File: simulator/electronic/controller/simulator/connection.kicad_sch (KiCad schematic)
At the start: 13 parts, among them J1 Conn_01x04_Socket, J1. Conn_01x04_Pin, J2 Conn_01x04_Socket, J2. Conn_01x04_Pin

Commit message: update simulator
Parts:
- removed D2: LED_DIR, LED_SMD:LED_RGB_5050-6, symbol Device:LED_RGB
- removed D3: LED_SW, LED_SMD:LED_RGB_5050-6, symbol Device:LED_RGB
- added D2: LED_UP, LED_SMD:LED_0805_2012Metric, symbol Device:LED
- added D3: LED_DOWN, LED_SMD:LED_0805_2012Metric, symbol Device:LED
- added D4: LED_BTM, LED_SMD:LED_0805_2012Metric, symbol Device:LED
- added D5: LED_CENTER, LED_SMD:LED_0805_2012Metric, symbol Device:LED
- added D6: LED_TOP, LED_SMD:LED_0805_2012Metric, symbol Device:LED
- renumbered J1. to J1.2, J2. to J2.2, R to R1, R5 to R4, R6 to R5, R7 to R6
Connections:
- net 3V3: now also D3.2 (A), D4.2 (A), D5.2 (A), D6.2 (A)
- net GND: now also D2.1 (K)
- net at R6.1: now also D6.1 (K)
- net at R4.1: now also D4.1 (K)
- net at R5.1: now also D5.1 (K)
- net at R2.1: now also D2.2 (A)
- net at R3.1: now also D3.1 (K)
Other:
- moved on the sheet: R2, R3, R4, R6

Commit message: update simulator
Parts:
- renumbered D6 to D2, D2 to D3, D5 to D4, D4 to D5, D3 to D6, J1.2 to J1.1, J2.2 to J2.1, R6 to R2, R2 to R3, R5 to R4, R4 to R5, R3 to R6

Commit message: update simulator
Parts:
- renumbered D3 to D2, D6 to D3, D2 to D4, D4 to D5, D5 to D6, R3 to R2, R6 to R3, R2 to R4, R4 to R5, R5 to R6

Commit message: update simulator
Parts:
- removed J1: Conn_01x04_Socket, Connector_Extra:JST_XH_B4B-XH-A_1x04_P2.54mm_Vertical, symbol Connector:Conn_01x04_Socket
- removed J1.1: Conn_01x04_Pin, symbol Connector:Conn_01x04_Pin
- added J1: Conn_01x03_Socket, Connector_JST:JST_XH_B3B-XH-A_1x03_P2.50mm_Vertical, symbol Connector:Conn_01x03_Socket
- added J1.1: Conn_01x03_Pin, symbol Connector:Conn_01x03_Pin
Connections:
- net DIR: now also J1.3 (Pin_3)
- net DIR_O: now also J1.1.3 (Pin_3)
- net GND: now also J1.1 (Pin_1); no longer D1.1 (K), D2.1 (K), J2.4 (Pin_4)
- net GND_O: now also J1.1.1 (Pin_1)
- net PULSE: now also J1.2 (Pin_2)
- net PULSE_O: now also J1.1.2 (Pin_2)
- new net: D1.1 (K), D2.1 (K), J2.4 (Pin_4)
Other:
- moved on the sheet: R1, R2, R3

Commit message: shaped schematic and PCB added printed documentation of PCB
Parts:
- R1, R2, R3, R4, R5, R6: value R_Small -> 150R
Connections:
- net GND: now also D1.1 (K), D2.1 (K), J2.4 (Pin_4)
Other:
- company: (none) -> HTL Leonding
- title: (none) -> Unseen-Obstacles - Simulator Controller

Commit message: finalized schematics and PCB
Connections:
- net GND_O: no longer J2.1.4 (Pin_4)
- new net SW_GND_O: J2.1.4 (Pin_4)
Changed lines of the file:
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@@
 		)
 	)
-	(hierarchical_label "GND_O"
+	(hierarchical_label "SW_GND_O"
 		(shape output)
 		(at 148.59 86.36 180)
